File: OpenAmigaFourPlayerAdapter.kicad_pcb (KiCad board)
At the start: 2 copper layers, 64.4 x 26.5 mm, 6 parts, among them J1 F25HP, J3 F09HP, J4 F09HP, J99 OSHW_LOGO

Commit message: 4 Player Adapter.* -> OpenAmigaFourPlayerAdapter.*
Parts:
- JP3, JP4: footprint 4 Player Adapter:PinHeader_1x02_P2.54mm_Vertical -> OpenAmigaFourPlayerAdapter:PinHeader_1x02_P2.54mm_Vertical
Changed lines of the file:
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@@
     )
   )
-  (module "4 Player Adapter:PinHeader_1x02_P2.54mm_Vertical" (layer Top)
+  (module OpenAmigaFourPlayerAdapter:PinHeader_1x02_P2.54mm_Vertical (layer Top)
     (at 123.6465 94.742)
     (descr "Through hole straight pin header, 1x02, 2.54mm pitch, single row")
@@
     )
   )
-  (module "4 Player Adapter:PinHeader_1x02_P2.54mm_Vertical" (layer Top)
+  (module OpenAmigaFourPlayerAdapter:PinHeader_1x02_P2.54mm_Vertical (layer Top)
     (at 157.195 94.742)
     (descr "Through hole straight pin header, 1x02, 2.54mm pitch, single row")
@@
   (segment (start 165.275 92.662) (end 165.275 94.742) (width 0.25) (layer Top) (net 9))
   (segment (start 165.275 99.211) (end 165.275 94.742) (width 0.25) (layer Bottom) (net 9))
-  (via (at 162.505 94.742) (size 0.6) (drill 0.4) (layers Top Bottom) (net 14))
-  (segment (start 162.505 89.2175) (end 162.505 92.7015) (width 0.25) (layer Top) (net 14) (status 10))
   (via (at 160.3855 108.5215) (size 0.6) (drill 0.4) (layers Top Bottom) (net 10))
   (segment (start 160.3855 111.6965) (end 160.3855 108.537) (width 0.25) (layer Top) (net 10) (status 10))
@@
   (via (at 150.642933 89.2175) (size 0.8) (drill 0.6) (layers Top Bottom) (net 13))
   (via (at 146.358566 89.2175) (size 0.8) (drill 0.6) (layers Top Bottom) (net 13))
+  (via (at 162.505 94.742) (size 0.6) (drill 0.4) (layers Top Bottom) (net 14))
+  (segment (start 162.505 89.2175) (end 162.505 92.7015) (width 0.25) (layer Top) (net 14) (status 10))
   (via (at 154.8455 106.8705) (size 0.6) (drill 0.4) (layers Top Bottom) (net 14))
   (segment (start 154.8455 106.8705) (end 154.8455 111.6965) (width 0.25) (layer Top) (net 14) (status 20))
